File: max1709/max1709.kicad_pcb (KiCad board)
At the start: 2 copper layers, 35 x 35 mm, 17 parts, among them U1 MAX1709

Commit message: complete
Parts:
- removed the REF** at (118.5, 78.5)
- removed the REF** at (146.5, 78.5)
- added REF**: MountingHole_2.2mm_M2, MountingHole:MountingHole_2.2mm_M2, F.Cu at (245.5, 104.0)
- added REF**: MountingHole_2.2mm_M2, MountingHole:MountingHole_2.2mm_M2, F.Cu at (204.5, 104.0)
- added SW1: SW_SPST, Connector_PinSocket_2.54mm:PinSocket_1x02_P2.54mm_Vertical, F.Cu at (204.5, 125.2)
- added TP1: VIN, Connector_PinSocket_2.54mm:PinSocket_1x01_P2.54mm_Vertical, F.Cu at (209.9, 103.8)
- added TP2: GND, Connector_PinSocket_2.54mm:PinSocket_1x01_P2.54mm_Vertical, F.Cu at (240.4, 103.8)
- added TP3: VOUT, Connector_PinSocket_2.54mm:PinSocket_1x01_P2.54mm_Vertical, F.Cu at (240.4, 115.8)
- D1: footprint Package_TO_SOT_SMD:TO-252-3_TabPin2 -> Package_TO_SOT_SMD:TO-252-2
- moved REF** 104.8 mm to (245.5, 141.0)
- moved REF** 95.8 mm to (225.0, 112.4)
- moved REF** 92.7 mm to (204.5, 141.0)
- moved C4 49.2 mm to (230.8, 133.8), turned to -90 degrees
- moved R1 45.7 mm to (209.2, 134.8)
- moved C2 44.9 mm to (214.6, 134.8)
- moved C1 44.7 mm to (211.9, 134.8)
- moved R2 43.8 mm to (227.2, 133.8), turned to -90 degrees
- moved C6 43.7 mm to (217.2, 108.5)
- moved C7 43.7 mm to (217.2, 115.0)
- moved D1 43.7 mm to (230.2, 119.5)
- moved L1 43.7 mm to (212.2, 121.0)
- moved U1 43.7 mm to (219.8, 128.5)
- moved C3 43.4 mm to (238.4, 124.5)
- moved C5 42.4 mm to (243.4, 124.5)
Connections:
- net /5v0 renamed Net-(C3-Pad1)
- net /VIN renamed Net-(C6-Pad1)
- U1 pad 1: unconnected-(U1-Pad1) -> Net-(U1-Pad1)
- U1 pad 12: (no net) -> Net-(C1-Pad1)
- U1 pad 6: Net-(C1-Pad1) -> Net-(D1-Pad3)
Routing:
- net Net-(C3-Pad1): track 0.00 -> 30.9 mm, vias 0 -> 2
- net Net-(C4-Pad1): track 0.00 -> 20.1 mm, vias 0 -> 2
- net Net-(U1-Pad1): track 0.00 -> 12.4 mm, vias 0 -> 2
- net GND: track 0.00 -> 10.6 mm
- net Net-(C1-Pad1): track 0.00 -> 8.48 mm
- net /VREF: track 0.00 -> 2.77 mm
- added copper zone on F.Cu, net GND
- added copper zone on F.Cu, net Net-(C3-Pad1)
- added copper zone on F.Cu, net Net-(C6-Pad1)
- added copper zone on F.Cu, net Net-(D1-Pad3)
Other:
- board size 35 x 35 mm -> 50 x 45 mm
- board text added: "JLCJLCJLCJLC"
