File: max1709/max1709.kicad_sch (KiCad schematic)
At the start: 12 parts, among them U1 MAX1709

Commit message: complete
Parts:
- added SW1: SW_SPST, Connector_PinSocket_2.54mm:PinSocket_1x02_P2.54mm_Vertical, symbol Switch:SW_SPST
- added TP1: VIN, Connector_PinSocket_2.54mm:PinSocket_1x01_P2.54mm_Vertical, symbol Connector:TestPoint
- added TP2: GND, Connector_PinSocket_2.54mm:PinSocket_1x01_P2.54mm_Vertical, symbol Connector:TestPoint
- added TP3: VOUT, Connector_PinSocket_2.54mm:PinSocket_1x01_P2.54mm_Vertical, symbol Connector:TestPoint
- D1: footprint Package_TO_SOT_SMD:TO-252-3_TabPin2 -> Package_TO_SOT_SMD:TO-252-2
Connections:
- net GND: now also SW1.1 (A), TP2.1
- net at U1.1 (ONA): now also SW1.2 (B)
- net at L1.1, U1.2 (LX), U1.3 (LX)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: now also D1.3 (A); no longer D1.2 (A)
- net at C1.1, R1.1: now also U1.12 (SS/LIM); no longer U1.6 (SS/LIM)
- net 5v0: no longer names the net of C3.1, C5.1, R2.2, U1.28 (ONB')
- net 5v0: now also D1.2 (K), TP3.1; no longer D1.1 (K)
- net VIN: no longer names the net of C6.1, C7.1, L1.2
- net VIN: now also TP1.1
Changed lines of the file:
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@@
   (junction (at 177.165 105.41) (diameter 0) (color 0 0 0 0))
   (junction (at 177.165 107.95) (diameter 0) (color 0 0 0 0))
+  (junction (at 179.07 107.95) (diameter 0) (color 0 0 0 0))
   (junction (at 180.975 90.17) (diameter 0) (color 0 0 0 0))
   (junction (at 180.975 115.57) (diameter 0) (color 0 0 0 0))
@@
   (junction (at 198.12 86.995) (diameter 0) (color 0 0 0 0))
   (no_connect (at 138.684 12.446))
-  (wire (pts (xy 114.3 66.04) (xy 120.65 66.04))
+  (wire (pts (xy 118.745 61.595) (xy 118.745 66.04))
+    (stroke (width 0) (type default) (color 0 0 0 0))
+  )
+  (wire (pts (xy 118.745 66.04) (xy 120.65 66.04))
     (stroke (width 0) (type default) (color 0 0 0 0))
   )
@@
     (stroke (width 0) (type default) (color 0 0 0 0))
   )
+  (wire (pts (xy 179.07 107.95) (xy 187.325 107.95))
+    (stroke (width 0) (type default) (color 0 0 0 0))
+  )
   (wire (pts (xy 180.975 90.17) (xy 180.975 87.63))
     (stroke (width 0) (type default) (color 0 0 0 0))
@@
   (wire (pts (xy 196.215 115.57) (xy 198.12 115.57))
     (stroke (width 0) (type default) (color 0 0 0 0))
-  )
-  (wire (pts (xy 198.12 74.295) (xy 199.39 74.295))
-    (stroke (width 0) (type solid) (color 0 0 0 0))
   )
   (wire (pts (xy 198.12 86.995) (xy 198.12 74.295))
@@
     (effects (font (size 1.27 1.27)) (justify left bottom))
   )
-  (label "VIN" (at 114.3 66.04 0)
-    (effects (font (size 1.27 1.27)) (justify left bottom))
-  )
   (label "VREF" (at 135.255 118.11 0)
     (effects (font (size 1.27 1.27)) (justify left bottom))
   )
-  (hierarchical_label "5v0" (shape output) (at 199.39 74.295 0)
-    (effects (font (size 1.27 1.27)) (justify left))
+  (symbol (lib_id "Connector:TestPoint") (at 118.745 61.595 0) (unit 1)
+    (in_bom yes) (on_board yes) (fields_autoplaced)
+    (property "Reference" "TP1" (id 0) (at 121.285 58.2929 0)
+      (effects (font (size 1.27 1.27)) (justify left))
+    )
+    (property "Value" "VIN" (id 1) (at 121.285 60.8329 0)
+      (effects (font (size 1.27 1.27)) (justify left))
+    )
+    (property "Footprint" "Connector_PinSocket_2.54mm:PinSocket_1x01_P2.54mm_Vertical" (id 2) (at 123.825 61.595 0)
+      (effects (font (size 1.27 1.27)) hide)
+    )
+    (property "Datasheet" "~" (id 3) (at 123.825 61.595 0)
+      (effects (font (size 1.27 1.27)) hide)
+    )
+    (pin "1")
+  )
+  (symbol (lib_id "Connector:TestPoint") (at 187.325 107.95 0) (unit 1)
+    (in_bom yes) (on_board yes) (fields_autoplaced)
+    (property "Reference" "TP2" (id 0) (at 189.23 104.6479 0)
+      (effects (font (size 1.27 1.27)) (justify left))
+    )
+    (property "Value" "GND" (id 1) (at 189.23 107.1879 0)
+      (effects (font (size 1.27 1.27)) (justify left))
+    )
+    (property "Footprint" "Connector_PinSocket_2.54mm:PinSocket_1x01_P2.54mm_Vertical" (id 2) (at 192.405 107.95 0)
+      (effects (font (size 1.27 1.27)) hide)
+    )
+    (property "Datasheet" "~" (id 3) (at 192.405 107.95 0)
+      (effects (font (size 1.27 1.27)) hide)
+    )
+    (pin "1")
+  )
+  (symbol (lib_id "Connector:TestPoint") (at 198.12 74.295 0) (unit 1)
+    (in_bom yes) (on_board yes) (fields_autoplaced)
+    (property "Reference" "TP3" (id 0) (at 200.025 70.9929 0)
+      (effects (font (size 1.27 1.27)) (justify left))
+    )
+    (property "Value" "VOUT" (id 1) (at 200.025 73.5329 0)
+      (effects (font (size 1.27 1.27)) (justify left))
+    )
+    (property "Footprint" "Connector_PinSocket_2.54mm:PinSocket_1x01_P2.54mm_Vertical" (id 2) (at 203.2 74.295 0)
+      (effects (font (size 1.27 1.27)) hide)
+    )
+    (property "Datasheet" "~" (id 3) (at 203.2 74.295 0)
+      (effects (font (size 1.27 1.27)) hide)
+    )
+    (pin "1")
   )
   (symbol (lib_id "power:GND") (at 120.65 73.66 0) (unit 1)
@@
     )
     (property "Datasheet" "" (id 3) (at 126.365 130.81 0)
+      (effects (font (size 1.27 1.27)) hide)
+    )
+    (pin "1")
+  )
+  (symbol (lib_id "power:GND") (at 136.525 85.09 0) (unit 1)
+    (in_bom yes) (on_board yes) (fields_autoplaced)
+    (property "Reference" "#PWR03" (id 0) (at 136.525 91.44 0)
+      (effects (font (size 1.27 1.27)) hide)
+    )
+    (property "Value" "GND" (id 1) (at 136.525 90.17 0))
+    (property "Footprint" "" (id 2) (at 136.525 85.09 0)
+      (effects (font (size 1.27 1.27)) hide)
+    )
+    (property "Datasheet" "" (id 3) (at 136.525 85.09 0)
       (effects (font (size 1.27 1.27)) hide)
     )
@@
   )
   (symbol (lib_id "Device:D_Schottky") (at 161.29 74.295 180) (unit 1)
-    (in_bom yes) (on_board yes) (fields_autoplaced)
-    (property "Reference" "D1" (id 0) (at 161.29 67.945 0))
-    (property "Value" "D_Schottky" (id 1) (at 161.29 70.485 0))
-    (property "Footprint" "Package_TO_SOT_SMD:TO-252-3_TabPin2" (id 2) (at 161.29 74.295 0)
+    (in_bom yes) (on_board yes)
+    (property "Reference" "D1" (id 0) (at 160.655 69.215 0))
+    (property "Value" "D_Schottky" (id 1) (at 161.29 71.755 0))
+    (property "Footprint" "Package_TO_SOT_SMD:TO-252-2" (id 2) (at 161.29 76.835 0)
       (effects (font (size 1.27 1.27)) hide)
     )
     (property "Datasheet" "~" (id 3) (at 161.29 74.295 0)
+      (effects (font (size 1.27 1.27)) hide)
+    )
+    (pin "2")
+    (pin "3")
+  )
+  (symbol (lib_id "Switch:SW_SPST") (at 141.605 85.09 0) (unit 1)
+    (in_bom yes) (on_board yes) (fields_autoplaced)
+    (property "Reference" "SW1" (id 0) (at 141.605 78.105 0))
+    (property "Value" "SW_SPST" (id 1) (at 141.605 80.645 0))
+    (property "Footprint" "Connector_PinSocket_2.54mm:PinSocket_1x02_P2.54mm_Vertical" (id 2) (at 141.605 85.09 0)
+      (effects (font (size 1.27 1.27)) hide)
+    )
+    (property "Datasheet" "~" (id 3) (at 141.605 85.09 0)
       (effects (font (size 1.27 1.27)) hide)
     )
@@
     (pin "1")
     (pin "11")
+    (pin "12")
     (pin "13")
     (pin "14")
@@
     (pin "5")
     (pin "6")
-    (pin "6")
     (pin "7")
     (pin "8")
@@
       (reference "#PWR02") (unit 1) (value "GND") (footprint "")
     )
+    (path "/d577914f-73ea-4516-ab9f-6c8c4e6485a7"
+      (reference "#PWR03") (unit 1) (value "GND") (footprint "")
+    )
     (path "/1138cc63-2807-493e-8ab5-2cec0c23206c"
       (reference "#PWR04") (unit 1) (value "GND") (footprint "")
@@
     )
     (path "/615f3d23-7399-4622-8cb4-41bb88dbebba"
-      (reference "D1") (unit 1) (value "D_Schottky") (footprint "Package_TO_SOT_SMD:TO-252-3_TabPin2")
+      (reference "D1") (unit 1) (value "D_Schottky") (footprint "Package_TO_SOT_SMD:TO-252-2")
     )
     (path "/92384637-e2d9-49e6-b68b-fa53f6f0f227"
@@
       (reference "R2") (unit 1) (value "2") (footprint "Resistor_SMD:R_1206_3216Metric_Pad1.30x1.75mm_HandSolder")
     )
+    (path "/4c7ad668-3412-4908-b940-3d5097bd77a8"
+      (reference "SW1") (unit 1) (value "SW_SPST") (footprint "Connector_PinSocket_2.54mm:PinSocket_1x02_P2.54mm_Vertical")
+    )
+    (path "/a024becb-b8a2-4831-a788-93bd5b39c678"
+      (reference "TP1") (unit 1) (value "VIN") (footprint "Connector_PinSocket_2.54mm:PinSocket_1x01_P2.54mm_Vertical")
+    )
+    (path "/8226fb32-d4ab-4a14-a8d2-63e9ab30b3be"
+      (reference "TP2") (unit 1) (value "GND") (footprint "Connector_PinSocket_2.54mm:PinSocket_1x01_P2.54mm_Vertical")
+    )
+    (path "/7bf0181c-d621-4e6f-bf55-f118649150c4"
+      (reference "TP3") (unit 1) (value "VOUT") (footprint "Connector_PinSocket_2.54mm:PinSocket_1x01_P2.54mm_Vertical")
+    )
     (path "/4987ec33-ac58-413a-83b3-f7438c6f0d8a"
